Commit message: feat: vla_control 추가 및 arm_bringup 설정 수정

File: vla_arm_ws/src/arm_bringup/urdf/panda_gazebo.urdf.xacro (robot description, xacro)
@@ -55,4 +55,7 @@
     <joint name="panda_joint7"><command_interface name="position"/><state_interface name="position"/><state_interface name="velocity"/></joint>
     <!-- 그리퍼(panda_finger_joint1/2)는 5-4 컨트롤러 설정과 함께 추가 예정 -->
+    <!-- 그리퍼: 열기(0.04m) ↔ 닫기(0.0m) 위치 제어 -->
+    <joint name="panda_finger_joint1"><command_interface name="position"/><state_interface name="position"/><state_interface name="velocity"/></joint>
+    <joint name="panda_finger_joint2"><command_interface name="position"/><state_interface name="position"/><state_interface name="velocity"/></joint>
   </ros2_control>
   <!-- gazebo_ros2_control 플러그인: 위 ros2_control 을 실제 컨트롤러(controllers.yaml)와 연결 -->
